File: xiao-stepper.kicad_pcb (KiCad board)
At the start: 2 copper layers, 42 x 42 mm, 20 parts, among them J1 Conn_PinHeader_1x04_P2.54mm_H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, M1 XIAO-RP2040_SocketSMD

Commit message: Updated PCB schematic
Parts:
- R1, R3: value 120 ohm -> 100 ohm
Changed lines of the file:
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@@
         (effects (font (size 1 1) (thickness 0.15)))
     )
-    (fp_text value "120 ohm" (at 0 1.9 90) (layer "F.Fab")
+    (fp_text value "100 ohm" (at 0 1.9 90) (layer "F.Fab")
         (effects (font (size 1 1) (thickness 0.15)))
     )
@@
         (effects (font (size 1 1) (thickness 0.15)))
     )
-    (fp_text value "120 ohm" (at 0 1.9) (layer "F.Fab")
-        (effects (font (size 1 1) (thickness 0.15)))
-    )
+    (fp_text value "100 ohm" (at 0 1.9) (layer "F.Fab")
+        (effects (font (size 1 1) (thickness 0.15)))
+    )
